Commit message: Add gazebo files

File: description/robot.urdf.xacro (robot description, xacro)
@@ -2,3 +2,4 @@
 <robot xmlns:xacro="http://www.ros.org/wiki/xacro"  name="robot">
   <xacro:include filename="robot_core.xacro"/>
+  <xacro:include filename="gazebo_control.xacro"/>
 </robot>

File: description/robot_core.xacro (robot description, xacro)
@@ -39,4 +39,7 @@
        </xacro:inertial_box>
    </link>
+   <gazebo reference="chassis_link">
+      <material>Gazebo/White</material>
+   </gazebo>
    <joint name="left_wheel_joint" type="continuous">
      <origin xyz="0 0.175 0" rpy="-${pi/2} 0 0"/>
@@ -63,4 +66,7 @@
       </xacro:inertial_cylinder>
    </link>
+    <gazebo reference="left_wheel_link">
+      <material>Gazebo/Blue</material>
+   </gazebo>
    <joint name="right_wheel_joint" type="continuous">
      <origin xyz="0 -0.175 0" rpy="${pi/2} 0 0"/>
@@ -87,4 +93,7 @@
       </xacro:inertial_cylinder>
    </link>
+   <gazebo reference="right_wheel_link">
+      <material>Gazebo/Blue</material>
+   </gazebo>
    <joint name="caster_wheel_joint" type="fixed">
      <origin xyz="0.24 0 0" rpy="0 0 0"/>
@@ -110,3 +119,8 @@
      </xacro:inertial_sphere>
    </link>
+   <gazebo reference="caster_wheel_link">
+      <material>Gazebo/Black</material>
+      <mu1 value="0.001"/>
+      <mu2 value="0.001"/>
+   </gazebo>
 </robot>

Commit message: add LIDAR for simulations

File: description/robot.urdf.xacro (robot description, xacro)
@@ -3,3 +3,4 @@
   <xacro:include filename="robot_core.xacro"/>
   <xacro:include filename="gazebo_control.xacro"/>
+  <xacro:include filename="lidar.xacro"/>
 </robot>

File: description/robot_core.xacro (robot description, xacro)
@@ -13,4 +13,7 @@
    <material name="black">
     <color rgba="0 0 0 1"/>
+   </material>
+   <material name="red">
+    <color rgba="1 0 0 1"/>
    </material>
    <link name="base_link">
@@ -81,5 +84,5 @@
            <cylinder length="0.04" radius="0.05"/>
         </geometry>
-        <material name="blue"/>;
+        <material name="blue"/>
       </visual>
       <collision>
