Commit message: Added slam tool functionality and ros2_control

File: description/lidar.xacro (robot description, xacro)
@@ -19,5 +19,5 @@
      <sensor name="laser" type="ray">
       <pose> 0 0 0 0 0 0 </pose>
-      <visualize>false</visualize>
+      <visualize>true</visualize>
       <update_rate>10</update_rate>
       <ray>

File: description/robot.urdf.xacro (robot description, xacro)
@@ -1,7 +1,12 @@
 <?xml version="1.0"?>
 <robot xmlns:xacro="http://www.ros.org/wiki/xacro"  name="robot">
+  <xacro:arg name="use_ros2_control" default="true"/>
   <xacro:include filename="robot_core.xacro"/>
-  <!-- <xacro:include filename="gazebo_control.xacro"/> -->
-  <xacro:include filename="ros2_control.xacro"/>
+  <xacro:if value="$(arg use_ros2_control)">
+    <xacro:include filename="ros2_control.xacro"/>
+  </xacro:if>
+  <xacro:unless value="$(arg use_ros2_control)">
+    <xacro:include filename="gazebo_control.xacro"/>
+  </xacro:unless>
   <xacro:include filename="lidar.xacro"/>
   <xacro:include filename="camera.xacro"/>

File: description/robot_core.xacro (robot description, xacro)
@@ -18,4 +18,11 @@
    </material>
    <link name="base_link">
+   </link>
+   <joint name="base_footprint_joint" type="fixed">
+      <origin xyz="0 0 0" rpy="0 0 0"/>
+      <parent link = "base_link"/>
+      <child link = "base_footprint"/>
+   </joint>
+   <link name="base_footprint">
    </link>
    <joint name="chassis_joint" type="fixed">
