Commit message: Added navigation, SLAM and OPEN-CV functionality

File: description/camera.xacro (robot description, xacro)
@@ -2,5 +2,5 @@
 <robot xmlns:xacro="http://www.ros.org/wiki/xacro">
   <joint name="camera_joint" type="fixed">
-    <origin xyz="0.305 0 0.08" rpy="0 0 0"/>
+    <origin xyz="0.305 0 0.08" rpy="0 0.18 0"/>
     <parent link = "chassis_link"/>
     <child link = "camera_link"/>

File: description/robot_core.xacro (robot description, xacro)
@@ -69,5 +69,5 @@
         <origin xyz="0 0 0" rpy="0 0 0"/>
         <geometry>
-           <cylinder length="0.04" radius="0.05"/>
+           <sphere radius="0.05"/>
         </geometry>
       </collision>
@@ -96,5 +96,5 @@
         <origin xyz="0 0 0" rpy="0 0 0"/>
         <geometry>
-           <cylinder length="0.04" radius="0.05"/>
+           <sphere radius="0.05"/>
         </geometry>
       </collision>
